Commit message: Step 2 Finshed

File: Step2/robotics_lab.urdf.xacro (robot description, xacro)
@@ -11,3 +11,15 @@
         <origin xyz="0 0 1" rpy="0 0 0" />
     </xacro:rrbot>
+    <xacro:table prefix="table_1" parent="world">
+        <origin xyz="0 10 0" rpy="0 0 0" />
+    </xacro:table>
+    <xacro:rrbot prefix="rrbot_1" parent="table_top">
+        <origin xyz="0 10 1" rpy="0 0 0" />
+    </xacro:rrbot>
+    <xacro:table prefix="table_2" parent="world">
+        <origin xyz="10 0 0" rpy="0 0 0" />
+    </xacro:table>
+    <xacro:rrbot prefix="rrbot_2" parent="table_top">
+        <origin xyz="10 0 1" rpy="0 0 0" />
+    </xacro:rrbot>
 </robot>

File: Step2/rrbot_macro.xacro (robot description, xacro)
@@ -6,5 +6,5 @@
     <xacro:property name="height0" value="2" /> <!-- base_link -->
     <xacro:property name="height1" value="1" /> <!-- link1 -->
-    <xacro:property name="height2" value="1" /> <!-- link2 -->
+    <xacro:property name="height2" value="2" /> <!-- link2 -->
     <xacro:property name="axel_offset" value="0.05" /> <!-- Space between top of beam and each joint -->
     <joint name="${prefix}base_joint" type="fixed">

File: Step2/table_on_rrbot.urdf.xacro (robot description, xacro)
@@ -9,5 +9,5 @@
     </xacro:rrbot>
     <xacro:table prefix="table_" parent="rrbot_tool0">
-        <origin xyz="0 0 0" rpy="${pi} 0 0" />
+        <origin xyz="0 0 0.975" rpy="${pi} 0 0" />
     </xacro:table>
 </robot>
