Commit message: Finshed Step 4

File: ws2/src/ur3e_on_table/urdf/ur3e_on_table.urdf.xacro (robot description, xacro)
@@ -5,5 +5,5 @@
     <link name="world" />
     <xacro:table prefix="table_" parent="world">
-        <origin xyz="0 0 1" rpy="0 0 0" />
+        <origin xyz="0 0 0" rpy="0 0 0" />
     </xacro:table>
     <!-- robot name parameter -->
@@ -42,5 +42,5 @@
         safety_k_position="$(arg safety_k_position)"
     >
-        <origin xyz="0 0 0" rpy="0 0 0" />          <!-- position robot in the world -->
+        <origin xyz="0 0 0.975" rpy="0 0 0" />          <!-- position robot in the world -->
     </xacro:ur_robot>
 </robot>
